Commit message: Add ros2_control for proper joint control
- ros2_control hardware interface in URDF
- Controller config (joint_state_broadcaster + joint_trajectory_controller)
- Updated launch file to spawn controllers
- Added ros2_controllers to Dockerfile

File: src/robot_description/urdf/robot.urdf.xacro (robot description, xacro)
@@ -261,24 +261,46 @@
     <material>Gazebo/Black</material>
   </gazebo>
-  <!-- Gazebo joint state publisher (publishes joint states FROM Gazebo) -->
+  <!-- ros2_control hardware interface -->
+  <ros2_control name="GazeboSystem" type="system">
+    <hardware>
+      <plugin>gazebo_ros2_control/GazeboSystem</plugin>
+    </hardware>
+    <joint name="shoulder_pan_joint">
+      <command_interface name="position">
+        <param name="min">-3.14</param>
+        <param name="max">3.14</param>
+      </command_interface>
+      <state_interface name="position"/>
+      <state_interface name="velocity"/>
+    </joint>
+    <joint name="shoulder_lift_joint">
+      <command_interface name="position">
+        <param name="min">-1.57</param>
+        <param name="max">1.57</param>
+      </command_interface>
+      <state_interface name="position"/>
+      <state_interface name="velocity"/>
+    </joint>
+    <joint name="elbow_joint">
+      <command_interface name="position">
+        <param name="min">-2.5</param>
+        <param name="max">2.5</param>
+      </command_interface>
+      <state_interface name="position"/>
+      <state_interface name="velocity"/>
+    </joint>
+    <joint name="wrist_joint">
+      <command_interface name="position">
+        <param name="min">-3.14</param>
+        <param name="max">3.14</param>
+      </command_interface>
+      <state_interface name="position"/>
+      <state_interface name="velocity"/>
+    </joint>
+  </ros2_control>
+  <!-- Gazebo ros2_control plugin -->
   <gazebo>
-    <plugin name="gazebo_ros_joint_state_publisher" filename="libgazebo_ros_joint_state_publisher.so">
-      <ros>
-        <namespace>/</namespace>
-      </ros>
-      <update_rate>50</update_rate>
-      <joint_name>shoulder_pan_joint</joint_name>
-      <joint_name>shoulder_lift_joint</joint_name>
-      <joint_name>elbow_joint</joint_name>
-      <joint_name>wrist_joint</joint_name>
-    </plugin>
-  </gazebo>
-  <!-- Gazebo joint pose trajectory (allows setting joint positions) -->
-  <gazebo>
-    <plugin name="gazebo_ros_joint_pose_trajectory" filename="libgazebo_ros_joint_pose_trajectory.so">
-      <ros>
-        <namespace>/</namespace>
-      </ros>
-      <update_rate>50</update_rate>
+    <plugin filename="libgazebo_ros2_control.so" name="gazebo_ros2_control">
+      <parameters>$(find robot_description)/config/controllers.yaml</parameters>
     </plugin>
   </gazebo>

Commit message: Fix camera orientation - point forward instead of down

File: src/robot_description/urdf/robot.urdf.xacro (robot description, xacro)
@@ -221,5 +221,5 @@
     <parent link="ee_link"/>
     <child link="camera_link"/>
-    <origin xyz="0.05 0 0" rpy="0 1.57 0"/>  <!-- Camera points forward/down -->
+    <origin xyz="0.05 0 0" rpy="0 0 0"/>  <!-- Camera points same direction as gripper -->
   </joint>
   <!-- Camera optical frame (Z forward, X right, Y down - standard camera convention) -->
